File: BBB-Cape-template/bbb-cape-template/bbb-cape-template.kicad_sch (KiCad schematic)
At the start: 11 parts, among them P8 BeagleBone_Black_Header, P9 BeagleBone_Black_Header, SW1 SW_DIP_x02, U1 CAT24C256

Commit message: added nor memory symbols
Parts:
- added IC1, IC2, IC3, IC4: IS25LP01GJ-RMLE-TY, SOIC127P1032X265-16N, symbol Memory Chip:IS25LP01GJ-RMLE-TY
