File: sheets/bbb_core.kicad_sch (KiCad schematic)
At the start: 0 parts

Commit message: Adding BBB cape and NOR flash ICs
Parts:
- added P10, P11: BeagleBone_Black_Header, Connector_PinHeader_2.54mm:PinHeader_2x23_P2.54mm_Vertical, symbol Connector_Generic:Conn_02x23_Odd_Even
- added R10, R11: 5.6k, symbol Device:R_Small
- added R12, R7, R8, R9: 10k, symbol Device:R_Small
- added SW2: SW_DIP_x02, symbol Switch:SW_DIP_x02
- added TP2: WP, symbol Connector:TestPoint
- added U2: CAT24C256, symbol Memory_EEPROM:CAT24C256
Connections:
- new net: R12.2, TP2.1, U2.7 (WP)
- new net: R8.2, SW2.3, U2.2 (A1)
- new net: R9.2, SW2.4, U2.1 (A0)
- new net: R7.2, U2.3 (A2)
- new net +1V8: P10.32 (Pin_32)
- new net +3V3: P10.3 (Pin_3), P10.4 (Pin_4), R10.1, R11.1, R12.1, R7.1, R8.1, R9.1, U2.8 (VCC)
- new net +5V: P10.5 (Pin_5), P10.6 (Pin_6)
- new net AIN0: P10.39 (Pin_39)
- new net AIN1: P10.40 (Pin_40)
- new net AIN2: P10.37 (Pin_37)
- new net AIN3: P10.38 (Pin_38)
- new net AIN4: P10.33 (Pin_33)
- new net AIN5: P10.36 (Pin_36)
- new net AIN6: P10.35 (Pin_35)
- new net GNDA: P10.34 (Pin_34)
- new net GNDD: P10.1 (Pin_1), P10.2 (Pin_2), P10.43 (Pin_43), P10.44 (Pin_44), P10.45 (Pin_45), P10.46 (Pin_46), P11.1 (Pin_1), P11.2 (Pin_2), SW2.1, SW2.2, U2.4 (GND)
- new net GPIO117: P10.25 (Pin_25)
- new net GPIO122: P10.30 (Pin_30)
- new net GPIO125: P10.27 (Pin_27)
- new net GPIO14: P10.26 (Pin_26)
- new net GPIO15: P10.24 (Pin_24)
- new net GPIO2: P10.22 (Pin_22)
- new net GPIO20: P10.41 (Pin_41)
- new net GPIO22: P11.19 (Pin_19)
- new net GPIO23: P11.13 (Pin_13)
- new net GPIO26: P11.14 (Pin_14)
- new net GPIO27: P11.17 (Pin_17)
- new net GPIO3: P10.21 (Pin_21)
- new net GPIO30: P10.11 (Pin_11)
- new net GPIO31: P10.13 (Pin_13)
- new net GPIO4: P10.17 (Pin_17)
- new net GPIO40: P10.14 (Pin_14)
- new net GPIO44: P11.12 (Pin_12)
- new net GPIO45: P11.11 (Pin_11)
- new net GPIO46: P11.16 (Pin_16)
- new net GPIO47: P11.15 (Pin_15)
- new net GPIO48: P10.15 (Pin_15)
- new net GPIO49: P10.23 (Pin_23)
- new net GPIO5: P10.18 (Pin_18)
- new net GPIO51: P10.16 (Pin_16)
- new net GPIO60: P10.12 (Pin_12)
- new net GPIO61: P11.28 (Pin_28)
- new net GPIO65: P11.18 (Pin_18)
- new net GPIO66: P11.7 (Pin_7)
- new net GPIO67: P11.8 (Pin_8)
- new net GPIO68: P11.10 (Pin_10)
- new net GPIO69: P11.9 (Pin_9)
- new net GPIO7: P10.42 (Pin_42)
- new net I2C2.SCL: P10.19 (Pin_19), R11.2, U2.6 (SCL)
- new net I2C2.SDA: P10.20 (Pin_20), R10.2, U2.5 (SDA)
- new net LCD.AC_BIAS_E: P11.30 (Pin_30)
- new net LCD.DATA0: P11.45 (Pin_45)
- new net LCD.DATA1: P11.46 (Pin_46)
- new net LCD.DATA10: P11.36 (Pin_36)
- new net LCD.DATA11: P11.34 (Pin_34)
- new net LCD.DATA12: P11.35 (Pin_35)
- new net LCD.DATA13: P11.33 (Pin_33)
- new net LCD.DATA14: P11.31 (Pin_31)
- new net LCD.DATA15: P11.32 (Pin_32)
- new net LCD.DATA2: P11.43 (Pin_43)
- new net LCD.DATA3: P11.44 (Pin_44)
- new net LCD.DATA4: P11.41 (Pin_41)
- new net LCD.DATA5: P11.42 (Pin_42)
- new net LCD.DATA6: P11.39 (Pin_39)
- new net LCD.DATA7: P11.40 (Pin_40)
- new net LCD.DATA8: P11.37 (Pin_37)
- new net LCD.DATA9: P11.38 (Pin_38)
- new net LCD.HSYNC: P11.29 (Pin_29)
- new net LCD.PCLK: P11.26 (Pin_26)
- new net LCD.VSYNC: P11.27 (Pin_27)
- new net MMC1.CLK: P11.21 (Pin_21)
- new net MMC1.CMD: P11.20 (Pin_20)
- new net MMC1.DAT0: P11.25 (Pin_25)
- new net MMC1.DAT1: P11.24 (Pin_24)
- new net MMC1.DAT2: P11.5 (Pin_5)
- new net MMC1.DAT3: P11.6 (Pin_6)
- new net MMC1.DAT4: P11.23 (Pin_23)
- new net MMC1.DAT5: P11.22 (Pin_22)
- new net MMC1.DAT6: P11.3 (Pin_3)
- new net MMC1.DAT7: P11.4 (Pin_4)
- new net PWR_BUT: P10.9 (Pin_9)
- new net SPI1.CS0: P10.28 (Pin_28)
- new net SPI1.D0: P10.29 (Pin_29)
- new net SPI1.SCLK: P10.31 (Pin_31)
- new net VBUS: P10.7 (Pin_7), P10.8 (Pin_8)
- new net ~{SYS_RESET}: P10.10 (Pin_10)
