File: sheets/power_distribution.kicad_sch (KiCad schematic)
At the start: 0 parts

Commit message: power distrubtion schematic, exact components tbd
Parts:
- added C1, C2: C_Polarized BULK, symbol Device:C_Polarized
- added D2: TBD, Diode_SMD:Nexperia_DSN1608-2_1.6x0.8mm, symbol Diode:PTVS5V0Z1USK
- added F1: Fuse, symbol Device:Fuse
- added FB1: FerriteBead, symbol Device:FerriteBead
Connections:
- new net +3V3_CDH: C2.1, FB1.2
- new net +3V3_EPS_IN: FB1.1
- new net +5V_CDH: C1.1, D2.1 (K), F1.2
- new net +5V_EPS_IN: F1.1
- new net GND: C1.2, C2.2, D2.2 (A)
