File: sheets/nor_flash.kicad_sch (KiCad schematic)
At the start: 4 parts, among them IC5 IS25LP01GJ-RMLE-TY, IC6 IS25LP01GJ-RMLE-TY, IC7 IS25LP01GJ-RMLE-TY, IC8 IS25LP01GJ-RMLE-TY

Commit message: pushing storage
Parts:
- removed IC5, IC6, IC7, IC8: IS25LP01GJ-RMLE-TY, SOIC127P1032X265-16N, symbol Memory Chip:IS25LP01GJ-RMLE-TY
Connections:
- no-connect marks 32 -> 0

Commit message: Adding BBB cape and NOR flash ICs
Parts:
- added IC5, IC6, IC7, IC8: IS25LP01GJ-RMLE-TY, SOIC127P1032X265-16N, symbol Memory Chip:IS25LP01GJ-RMLE-TY

Commit message: push
Connections:
- net +3.3V: now reaches IC6.1 (HOLD#_OR_RESET#_(IO3))
- net +3.3V: now also IC5.1 (HOLD#_OR_RESET#_(IO3)), IC5.2 (VCC), IC5.9 (WP#_(IO2)), IC6.2 (VCC), IC6.9 (WP#_(IO2)), IC7.1 (HOLD#_OR_RESET#_(IO3)), IC7.2 (VCC), IC7.9 (WP#_(IO2)), IC8.1 (HOLD#_OR_RESET#_(IO3)), IC8.2 (VCC), IC8.9 (WP#_(IO2))
- net GNDD: now reaches IC6.10 (GND)
- net GNDD: now also IC5.10 (GND), IC7.10 (GND), IC8.10 (GND)
- net SPI0.D1: now reaches IC6.15 (SI_(IO0))
- net SPI0.D1: now also IC5.15 (SI_(IO0)), IC7.15 (SI_(IO0)), IC8.15 (SI_(IO0))
- net SPI0.SCLK: now reaches IC6.16 (SCK)
- net SPI0.SCLK: now also IC5.16 (SCK), IC7.16 (SCK), IC8.16 (SCK)
- net SPI0.CS1: now reaches IC6.7 (CE#)
- net SPI0.D0: now reaches IC6.8 (SO_(IO1))
- net SPI0.D0: now also IC5.8 (SO_(IO1)), IC7.8 (SO_(IO1)), IC8.8 (SO_(IO1))
- net SPI0.CS0: now reaches IC5.7 (CE#)
- net SPI0.CS3: now reaches IC8.7 (CE#)
- net SPI0.CS2: now reaches IC7.7 (CE#)
