File: sheets/pc104_interface.kicad_sch (KiCad schematic)
At the start: 0 parts

Commit message: CDH Updated to have Payload USB interface and Trigger connectors
Parts:
- added H1, H2, H3, H4: MountingHole_Pad, MountingHole:MountingHole_3.2mm_M3_Pad, symbol Mechanical:MountingHole_Pad
- added J3, J4: Conn_02x26_Row_Letter_First, Connector_PinSocket_2.54mm:PinSocket_2x26_P2.54mm_Vertical, symbol Connector_Generic:Conn_02x26_Row_Letter_First
Connections:
- new net 12V_out: J4.a12 (Pin_a12), J4.b12 (Pin_b12)
- new net 3V3_out: J4.a14 (Pin_a14), J4.b14 (Pin_b14)
- new net 5V_out: J3.a13 (Pin_a13), J3.b13 (Pin_b13), J4.a13 (Pin_a13), J4.b13 (Pin_b13)
- new net ACDS_IMU_RST: J3.b15 (Pin_b15)
- new net ACDS_PERM_5: J3.a15 (Pin_a15)
- new net ACDS_PERM_6: J3.a16 (Pin_a16)
- new net ACDS_PWM_1: J3.a9 (Pin_a9)
- new net ACDS_PWM_2: J3.a10 (Pin_a10)
- new net ACDS_PWM_3: J3.a11 (Pin_a11)
- new net ACDS_PWM_4: J3.a12 (Pin_a12)
- new net ACDS_RS232_RX: J3.b4 (Pin_b4)
- new net ACDS_RS232_TX: J3.b3 (Pin_b3)
- new net CM_SCL: J3.b9 (Pin_b9)
- new net CM_SDA: J3.b8 (Pin_b8)
- new net DS_A: J4.a26 (Pin_a26)
- new net DS_B: J4.b26 (Pin_b26)
- new net GND: H1.1, H2.1, H3.1, H4.1, J3.a17 (Pin_a17), J3.b17 (Pin_b17), J4.a15 (Pin_a15), J4.a16 (Pin_a16), J4.b15 (Pin_b15), J4.b16 (Pin_b16)
- new net HEATER_PWM: J4.b10 (Pin_b10)
- new net INT: J3.b6 (Pin_b6)
- new net PG: J3.b5 (Pin_b5)
- new net RBF_A: J4.a25 (Pin_a25)
- new net RBF_B: J4.b25 (Pin_b25)
- new net RS SYS2 Rx: J3.a20 (Pin_a20)
- new net RS SYS2 Tx: J3.b20 (Pin_b20)
- new net RS-485 SYS1 A: J3.b12 (Pin_b12)
- new net RS-485 SYS1 B: J3.b11 (Pin_b11)
- new net SOL_PIN: J4.a22 (Pin_a22), J4.b22 (Pin_b22)
- new net STAT_1: J3.b7 (Pin_b7)
- new net STAT_2: J3.a5 (Pin_a5)
- new net SUN_SENSE_1: J4.a1 (Pin_a1)
- new net SUN_SENSE_2: J4.b1 (Pin_b1)
- new net SUN_SENSE_3: J4.a2 (Pin_a2)
- new net SUN_SENSE_4: J4.b2 (Pin_b2)
- new net SYS_PIN: J4.b23 (Pin_b23), J4.b24 (Pin_b24)
- new net THR_1: J4.a3 (Pin_a3)
- new net THR_2: J4.b3 (Pin_b3)
- new net THR_3: J4.a4 (Pin_a4)
- new net THR_4: J4.b4 (Pin_b4)
- new net THR_5: J4.b5 (Pin_b5)
- new net THR_6: J4.b6 (Pin_b6)
- new net THR_7: J4.b7 (Pin_b7)
- new net THR_8: J4.b8 (Pin_b8)
- new net THR_9: J4.b9 (Pin_b9)
- new net UART_RX: J3.b21 (Pin_b21)
- new net UART_TX: J3.b22 (Pin_b22)
- new net V_Batt: J4.a23 (Pin_a23), J4.a24 (Pin_a24)
- no-connect marks 0 -> 45

Commit message: Payload USB updated to have 4 USB 2.0 Hub
Added support for USB flash or eUSB flash for storage.
Parts:
- renumbered J3 to J1, J4 to J2
Changed lines of the file:
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@@
 		(dnp no)
 		(fields_autoplaced yes)
-		(property "Reference" "#PWR020"
+		(property "Reference" "#PWR034"
 			(at 156.21 38.1 0)
 			(hide yes)
@@
 			(project "hs2-cdh-pcb"
 				(path "/e63e39d7-6ac0-4ffd-8aa3-1841a4541b55/b0136f55-db06-4889-9369-30a271664d5f"
-					(reference "#PWR020")
+					(reference "#PWR034")
 					(unit 1)
 				)
@@
 		(dnp no)
 		(fields_autoplaced yes)
-		(property "Reference" "#PWR018"
+		(property "Reference" "#PWR033"
 			(at 127.4093 72.2977 0)
 			(hide yes)
@@
 			(project "hs2-cdh-pcb"
 				(path "/e63e39d7-6ac0-4ffd-8aa3-1841a4541b55/b0136f55-db06-4889-9369-30a271664d5f"
-					(reference "#PWR018")
+					(reference "#PWR033")
 					(unit 1)
 				)
@@
 		(dnp no)
 		(fields_autoplaced yes)
-		(property "Reference" "#PWR022"
+		(property "Reference" "#PWR036"
 			(at 156.21 66.04 0)
 			(hide yes)
@@
 			(project "hs2-cdh-pcb"
 				(path "/e63e39d7-6ac0-4ffd-8aa3-1841a4541b55/b0136f55-db06-4889-9369-30a271664d5f"
-					(reference "#PWR022")
+					(reference "#PWR036")
 					(unit 1)
 				)
@@
 		(dnp no)
 		(fields_autoplaced yes)
-		(property "Reference" "#PWR014"
+		(property "Reference" "#PWR031"
 			(at 57.15 73.66 0)
 			(hide yes)
@@
 			(project "hs2-cdh-pcb"
 				(path "/e63e39d7-6ac0-4ffd-8aa3-1841a4541b55/b0136f55-db06-4889-9369-30a271664d5f"
-					(reference "#PWR014")
+					(reference "#PWR031")
 					(unit 1)
 				)
@@
 		(dnp no)
 		(fields_autoplaced yes)
-		(property "Reference" "J3"
+		(property "Reference" "J1"
 			(at 45.72 20.0898 0)
 			(show_name no)
@@
 			(project "hs2-cdh-pcb"
 				(path "/e63e39d7-6ac0-4ffd-8aa3-1841a4541b55/b0136f55-db06-4889-9369-30a271664d5f"
-					(reference "J3")
+					(reference "J1")
 					(unit 1)
 				)
@@
 		(dnp no)
 		(fields_autoplaced yes)
-		(property "Reference" "#PWR023"
+		(property "Reference" "#PWR037"
 			(at 156.21 80.01 0)
 			(hide yes)
@@
 			(project "hs2-cdh-pcb"
 				(path "/e63e39d7-6ac0-4ffd-8aa3-1841a4541b55/b0136f55-db06-4889-9369-30a271664d5f"
-					(reference "#PWR023")
+					(reference "#PWR037")
 					(unit 1)
 				)
@@
 		(dnp no)
 		(fields_autoplaced yes)
-		(property "Reference" "#PWR021"
+		(property "Reference" "#PWR035"
 			(at 156.21 52.07 0)
 			(hide yes)
@@
 			(project "hs2-cdh-pcb"
 				(path "/e63e39d7-6ac0-4ffd-8aa3-1841a4541b55/b0136f55-db06-4889-9369-30a271664d5f"
-					(reference "#PWR021")
+					(reference "#PWR035")
 					(unit 1)
 				)
@@
 		(dnp no)
 		(fields_autoplaced yes)
-		(property "Reference" "#PWR09"
+		(property "Reference" "#PWR030"
 			(at 34.29 73.66 0)
 			(hide yes)
@@
 			(project "hs2-cdh-pcb"
 				(path "/e63e39d7-6ac0-4ffd-8aa3-1841a4541b55/b0136f55-db06-4889-9369-30a271664d5f"
-					(reference "#PWR09")
+					(reference "#PWR030")
 					(unit 1)
 				)
@@
 		(dnp no)
 		(fields_autoplaced yes)
-		(property "Reference" "J4"
+		(property "Reference" "J2"
 			(at 114.3 20.9963 0)
 			(show_name no)
@@
 			(project "hs2-cdh-pcb"
 				(path "/e63e39d7-6ac0-4ffd-8aa3-1841a4541b55/b0136f55-db06-4889-9369-30a271664d5f"
-					(reference "J4")
+					(reference "J2")
 					(unit 1)
 				)
@@
 		(dnp no)
 		(fields_autoplaced yes)
-		(property "Reference" "#PWR015"
+		(property "Reference" "#PWR032"
 			(at 102.0488 72.2213 0)
 			(hide yes)
@@
 			(project "hs2-cdh-pcb"
 				(path "/e63e39d7-6ac0-4ffd-8aa3-1841a4541b55/b0136f55-db06-4889-9369-30a271664d5f"
-					(reference "#PWR015")
+					(reference "#PWR032")
 					(unit 1)
 				)
