File: sheets/pc104_interface.kicad_sch (KiCad schematic)
At the start: 0 parts

Commit message: adding pc104 from EPS
Parts:
- added H1, H2, H3, H4: MountingHole_Pad, MountingHole:MountingHole_3.2mm_M3_Pad, symbol Mechanical:MountingHole_Pad
- added J3, J4: Conn_02x26_Row_Letter_First, Connector_PinSocket_2.54mm:PinSocket_2x26_P2.54mm_Vertical, symbol Connector_Generic:Conn_02x26_Row_Letter_First
Connections:
- new net 12V: J4.a12 (Pin_a12), J4.b12 (Pin_b12)
- new net 3.3V: J4.a14 (Pin_a14), J4.b14 (Pin_b14)
- new net 5V_PERM: J3.a13 (Pin_a13), J3.b13 (Pin_b13), J4.a13 (Pin_a13), J4.b13 (Pin_b13)
- new net ACDS_GPIO_1: J3.a10 (Pin_a10)
- new net ACDS_GPIO_2: J3.a12 (Pin_a12)
- new net ACDS_GPIO_3: J3.a16 (Pin_a16)
- new net ACDS_IMU_RST: J3.b15 (Pin_b15)
- new net ACDS_PWM_1: J3.a9 (Pin_a9)
- new net ACDS_PWM_2: J3.a11 (Pin_a11)
- new net ACDS_PWM_3: J3.a15 (Pin_a15)
- new net ACDS_RS232_RX: J3.b4 (Pin_b4)
- new net ACDS_RS232_TX: J3.b3 (Pin_b3)
- new net BATT_PIN: J4.a23 (Pin_a23), J4.a24 (Pin_a24)
- new net DS_A: J4.a26 (Pin_a26)
- new net DS_B: J4.b26 (Pin_b26)
- new net GND: H1.1, H2.1, H3.1, H4.1, J3.a17 (Pin_a17), J3.b17 (Pin_b17), J4.a15 (Pin_a15), J4.a16 (Pin_a16), J4.b15 (Pin_b15), J4.b16 (Pin_b16)
- new net HEATER_PWM: J4.b10 (Pin_b10)
- new net INT: J3.b6 (Pin_b6)
- new net PG: J3.b5 (Pin_b5)
- new net RBF_A: J4.a25 (Pin_a25)
- new net RBF_B: J4.b25 (Pin_b25)
- new net RS SYS2 Rx: J3.a20 (Pin_a20)
- new net RS SYS2 Tx: J3.b20 (Pin_b20)
- new net RS-485 SYS1 A: J3.b12 (Pin_b12)
- new net RS-485 SYS1 B: J3.b11 (Pin_b11)
- new net SCL: J3.b9 (Pin_b9)
- new net SDA: J3.b8 (Pin_b8)
- new net SOL_PIN: J4.a22 (Pin_a22), J4.b22 (Pin_b22)
- new net STAT_1: J3.b7 (Pin_b7)
- new net STAT_2: J3.a5 (Pin_a5)
- new net SUN_SENSE_1: J4.a1 (Pin_a1)
- new net SUN_SENSE_2: J4.b1 (Pin_b1)
- new net SUN_SENSE_3: J4.a2 (Pin_a2)
- new net SUN_SENSE_4: J4.b2 (Pin_b2)
- new net SYS_PIN: J4.b23 (Pin_b23), J4.b24 (Pin_b24)
- new net THR_1: J4.a3 (Pin_a3)
- new net THR_2: J4.b3 (Pin_b3)
- new net THR_3: J4.a4 (Pin_a4)
- new net THR_4: J4.b4 (Pin_b4)
- new net THR_5: J4.b5 (Pin_b5)
- new net THR_6: J4.b6 (Pin_b6)
- new net THR_7: J4.b7 (Pin_b7)
- new net THR_8: J4.b8 (Pin_b8)
- new net THR_9: J4.b9 (Pin_b9)
- new net UART_RX: J3.b21 (Pin_b21)
- new net UART_TX: J3.b22 (Pin_b22)
- no-connect marks 0 -> 42

Commit message: allocating pins ?
Connections:
- net HEATER_PWM: now also J4.b21 (Pin_b21); no longer J4.b10 (Pin_b10)
- net THR_TC7_T+: now reaches J4.a10 (Pin_a10)
- net THR_TC8_T+: now reaches J4.a11 (Pin_a11)
- net THR_TC2_T+: now reaches J4.a5 (Pin_a5)
- net THR_TC3_T+: now reaches J4.a6 (Pin_a6)
- net THR_TC4_T+: now reaches J4.a7 (Pin_a7)
- net THR_TC5_T+: now reaches J4.a8 (Pin_a8)
- net THR_TC6_T+: now reaches J4.a9 (Pin_a9)
- net THR_TC8_T-: now reaches J4.b11 (Pin_b11)
- net SUN_SENSE_1 renamed SUN_SENS1_CH
- net SUN_SENSE_2 renamed SUN_SENS2_CH
- net SUN_SENSE_3 renamed SUN_SENS3_CH
- net SUN_SENSE_4 renamed SUN_SENS4_CH
- net THR_1 renamed SUN_SENS5_CH
- net THR_2 renamed SUN_SENS6_CH
- net THR_3 renamed THR_TC1_T+
- net THR_4 renamed THR_TC1_T-
- net THR_5 renamed THR_TC2_T-
- net THR_6 renamed THR_TC3_T-
- net THR_7 renamed THR_TC4_T-
- net THR_8 renamed THR_TC5_T-
- net THR_9 renamed THR_TC6_T-
- new net THR_TC7_T-: J4.b10 (Pin_b10)
- no-connect marks 42 -> 36

Commit message: Merge Payload and thermals
Parts:
- renumbered J3 to J1, J4 to J2
Changed lines of the file:
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@@
 		(dnp no)
 		(fields_autoplaced yes)
-		(property "Reference" "#PWR091"
+		(property "Reference" "#PWR042"
 			(at 109.22 95.25 0)
 			(hide yes)
@@
 			(project "hs2-cdh-pcb"
 				(path "/e63e39d7-6ac0-4ffd-8aa3-1841a4541b55/b0136f55-db06-4889-9369-30a271664d5f"
-					(reference "#PWR091")
+					(reference "#PWR042")
 					(unit 1)
 				)
@@
 		(dnp no)
 		(fields_autoplaced yes)
-		(property "Reference" "#PWR094"
+		(property "Reference" "#PWR045"
 			(at 198.12 62.23 0)
 			(hide yes)
@@
 			(project "hs2-cdh-pcb"
 				(path "/e63e39d7-6ac0-4ffd-8aa3-1841a4541b55/b0136f55-db06-4889-9369-30a271664d5f"
-					(reference "#PWR094")
+					(reference "#PWR045")
 					(unit 1)
 				)
@@
 		(dnp no)
 		(fields_autoplaced yes)
-		(property "Reference" "J3"
+		(property "Reference" "J1"
 			(at 96.52 41.6798 0)
 			(show_name no)
@@
 			(project "hs2-cdh-pcb"
 				(path "/e63e39d7-6ac0-4ffd-8aa3-1841a4541b55/b0136f55-db06-4889-9369-30a271664d5f"
-					(reference "J3")
+					(reference "J1")
 					(unit 1)
 				)
@@
 		(dnp no)
 		(fields_autoplaced yes)
-		(property "Reference" "J4"
+		(property "Reference" "J2"
 			(at 151.13 43.8563 0)
 			(show_name no)
@@
 			(project "hs2-cdh-pcb"
 				(path "/e63e39d7-6ac0-4ffd-8aa3-1841a4541b55/b0136f55-db06-4889-9369-30a271664d5f"
-					(reference "J4")
+					(reference "J2")
 					(unit 1)
 				)
@@
 		(in_pos_files yes)
 		(dnp no)
-		(property "Reference" "#PWR093"
+		(property "Reference" "#PWR044"
 			(at 165.1 93.98 0)
 			(hide yes)
@@
 			(project "hs2-cdh-pcb"
 				(path "/e63e39d7-6ac0-4ffd-8aa3-1841a4541b55/b0136f55-db06-4889-9369-30a271664d5f"
-					(reference "#PWR093")
+					(reference "#PWR044")
 					(unit 1)
 				)
@@
 		(dnp no)
 		(fields_autoplaced yes)
-		(property "Reference" "#PWR095"
+		(property "Reference" "#PWR046"
 			(at 198.12 76.2 0)
 			(hide yes)
@@
 			(project "hs2-cdh-pcb"
 				(path "/e63e39d7-6ac0-4ffd-8aa3-1841a4541b55/b0136f55-db06-4889-9369-30a271664d5f"
-					(reference "#PWR095")
+					(reference "#PWR046")
 					(unit 1)
 				)
@@
 		(in_pos_files yes)
 		(dnp no)
-		(property "Reference" "#PWR092"
+		(property "Reference" "#PWR043"
 			(at 138.43 93.98 0)
 			(hide yes)
@@
 			(project "hs2-cdh-pcb"
 				(path "/e63e39d7-6ac0-4ffd-8aa3-1841a4541b55/b0136f55-db06-4889-9369-30a271664d5f"
-					(reference "#PWR092")
+					(reference "#PWR043")
 					(unit 1)
 				)
@@
 		(dnp no)
 		(fields_autoplaced yes)
-		(property "Reference" "#PWR090"
+		(property "Reference" "#PWR041"
 			(at 82.55 95.25 0)
 			(hide yes)
@@
 			(project "hs2-cdh-pcb"
 				(path "/e63e39d7-6ac0-4ffd-8aa3-1841a4541b55/b0136f55-db06-4889-9369-30a271664d5f"
-					(reference "#PWR090")
+					(reference "#PWR041")
 					(unit 1)
 				)
@@
 		(dnp no)
 		(fields_autoplaced yes)
-		(property "Reference" "#PWR096"
+		(property "Reference" "#PWR047"
 			(at 198.12 90.17 0)
 			(hide yes)
@@
 			(project "hs2-cdh-pcb"
 				(path "/e63e39d7-6ac0-4ffd-8aa3-1841a4541b55/b0136f55-db06-4889-9369-30a271664d5f"
-					(reference "#PWR096")
+					(reference "#PWR047")
 					(unit 1)
 				)
@@
 		(dnp no)
 		(fields_autoplaced yes)
-		(property "Reference" "#PWR097"
+		(property "Reference" "#PWR048"
 			(at 198.12 104.14 0)
 			(hide yes)
@@
 			(project "hs2-cdh-pcb"
 				(path "/e63e39d7-6ac0-4ffd-8aa3-1841a4541b55/b0136f55-db06-4889-9369-30a271664d5f"
-					(reference "#PWR097")
-					(unit 1)
-				)
+					(reference "#PWR048")
+					(unit 1)
+				)
