File: sheets/adcs_sun_adc.kicad_sch (KiCad schematic)
At the start: 1 part, among them U10 MCP3208

Commit message: push
Parts:
- added C13, C14: 0.1uF, symbol Device:C
Connections:
- net SUN1_CH: now reaches U10.1 (CH0)
- net SPI1.CS0: now reaches U10.10 (~{CS}/SHDN)
- net SPI1.D1: now reaches U10.11 (Din)
- net SPI1.D0: now reaches U10.12 (Dout)
- net SPI1.SCLK: now reaches U10.13 (CLK)
- net GNDA: now reaches U10.14 (AGND)
- net GNDA: now also C14.2
- net +3.3V: now reaches U10.15 (Vref)
- net +3.3V: now also U10.16 (Vdd), C13.1, C14.1
- net SUN2_CH: now reaches U10.2 (CH1)
- net SUN3_CH: now reaches U10.3 (CH2)
- net SUN4_CH: now reaches U10.4 (CH3)
- net SUN5_CH: now reaches U10.5 (CH4)
- net SUN6_CH: now reaches U10.6 (CH5)
- net GNDD: now reaches U10.9 (DGND)
- net GNDD: now also C13.2
- no-connect marks 0 -> 2

Commit message: allocating pins ?
Connections:
- net SUN1_CH renamed SUN_SENS1_CH
- net SUN2_CH renamed SUN_SENS2_CH
- net SUN3_CH renamed SUN_SENS3_CH
- net SUN4_CH renamed SUN_SENS4_CH
- net SUN5_CH renamed SUN_SENS5_CH
- net SUN6_CH renamed SUN_SENS6_CH
Changed lines of the file:
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@@
 		)
 	)
-	(global_label "SUN4_CH"
+	(global_label "SUN_SENS4_CH"
 		(shape input)
 		(at 133.35 91.44 180)
@@
 		)
 		(property "Intersheetrefs" "${INTERSHEET_REFS}"
-			(at 121.6216 91.44 0)
-			(hide yes)
-			(show_name no)
-			(do_not_autoplace no)
-			(effects
-				(font
-					(size 1.27 1.27)
-				)
-				(justify right)
-			)
-		)
-	)
-	(global_label "SUN6_CH"
+			(at 115.7555 91.44 0)
+			(hide yes)
+			(show_name no)
+			(do_not_autoplace no)
+			(effects
+				(font
+					(size 1.27 1.27)
+				)
+				(justify right)
+			)
+		)
+	)
+	(global_label "SUN_SENS6_CH"
 		(shape input)
 		(at 133.35 96.52 180)
@@
 		)
 		(property "Intersheetrefs" "${INTERSHEET_REFS}"
-			(at 121.6216 96.52 0)
-			(hide yes)
-			(show_name no)
-			(do_not_autoplace no)
-			(effects
-				(font
-					(size 1.27 1.27)
-				)
-				(justify right)
-			)
-		)
-	)
-	(global_label "SUN2_CH"
+			(at 115.7555 96.52 0)
+			(hide yes)
+			(show_name no)
+			(do_not_autoplace no)
+			(effects
+				(font
+					(size 1.27 1.27)
+				)
+				(justify right)
+			)
+		)
+	)
+	(global_label "SUN_SENS2_CH"
 		(shape input)
 		(at 133.35 86.36 180)
@@
 		)
 		(property "Intersheetrefs" "${INTERSHEET_REFS}"
-			(at 121.6216 86.36 0)
+			(at 115.7555 86.36 0)
 			(hide yes)
 			(show_name no)
@@
 		)
 	)
-	(global_label "SUN3_CH"
+	(global_label "SUN_SENS3_CH"
 		(shape input)
 		(at 133.35 88.9 180)
@@
 		)
 		(property "Intersheetrefs" "${INTERSHEET_REFS}"
-			(at 121.6216 88.9 0)
-			(hide yes)
-			(show_name no)
-			(do_not_autoplace no)
-			(effects
-				(font
-					(size 1.27 1.27)
-				)
-				(justify right)
-			)
-		)
-	)
-	(global_label "SUN5_CH"
+			(at 115.7555 88.9 0)
+			(hide yes)
+			(show_name no)
+			(do_not_autoplace no)
+			(effects
+				(font
+					(size 1.27 1.27)
+				)
+				(justify right)
+			)
+		)
+	)
+	(global_label "SUN_SENS5_CH"
 		(shape input)
 		(at 133.35 93.98 180)
@@
 		)
 		(property "Intersheetrefs" "${INTERSHEET_REFS}"
-			(at 121.6216 93.98 0)
+			(at 115.7555 93.98 0)
 			(hide yes)
 			(show_name no)
@@
 		)
 	)
-	(global_label "SUN1_CH"
+	(global_label "SUN_SENS1_CH"
 		(shape input)
 		(at 133.35 83.82 180)
@@
 		)
 		(property "Intersheetrefs" "${INTERSHEET_REFS}"
-			(at 121.6216 83.82 0)
-			(hide yes)
-			(show_name no)
+			(at 115.7555 83.82 0)
+			(hide yes)
+			(show_name no)

Commit message: ferrite bead
Parts:
- added FB3: FerriteBead, symbol Device:FerriteBead
Connections:
- net +3.3V: now also FB3.1; no longer C14.1, U10.15 (Vref)
- new net: C14.1, FB3.2, U10.15 (Vref)
Changed lines of the file:
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@@
 	(paper "A4")
+	(junction
+		(at 153.67 62.23)
+		(diameter 0)
+		(color 0 0 0 0)
+	)
 	(junction
 		(at 146.05 62.23)
@@
 		(color 0 0 0 0)
 	)
-	(junction
-		(at 153.67 62.23)
-		(diameter 0)
-		(color 0 0 0 0)
-	)
 	(no_connect
 		(at 133.35 99.06)
@@
 		(pts
 			(xy 146.05 62.23) (xy 146.05 78.74)
-		)
-		(stroke
-			(width 0)
-			(type default)
-		)
-	)
-	(wire
-		(pts
-			(xy 146.05 60.96) (xy 146.05 62.23)
 		)
 		(stroke
@@
 	(symbol
 		(lib_id "power:+3.3V")
-		(at 146.05 60.96 0)
+		(at 146.05 54.61 0)
 		(unit 1)
 		(body_style 1)
@@
 		(fields_autoplaced yes)
 		(property "Reference" "#PWR040"
-			(at 146.05 64.77 0)
+			(at 146.05 58.42 0)
 			(hide yes)
 			(show_name no)
@@
 		)
 		(property "Value" "+3.3V"
-			(at 146.05 55.88 0)
+			(at 146.05 49.53 0)
 			(show_name no)
 			(do_not_autoplace no)
@@
 		)
 		(property "Footprint" ""
-			(at 146.05 60.96 0)
+			(at 146.05 54.61 0)
 			(hide yes)
 			(show_name no)
@@
 		)
 		(property "Datasheet" ""
-			(at 146.05 60.96 0)
+			(at 146.05 54.61 0)
 			(hide yes)
 			(show_name no)
@@
 		)
 		(property "Description" "Power symbol creates a global label with name \"+3.3V\""
-			(at 146.05 60.96 0)
+			(at 146.05 54.61 0)
 			(hide yes)
 			(show_name no)
@@
 					(unit 1)
 				)
+			)
+		)
+	)
+	(symbol
+		(lib_id "Device:FerriteBead")
+		(at 146.05 58.42 0)
+		(unit 1)
+		(body_style 1)
+		(exclude_from_sim no)
+		(in_bom yes)
+		(on_board yes)
+		(in_pos_files yes)
+		(dnp no)
+		(property "Reference" "FB3"
+			(at 132.588 56.896 0)
+			(show_name no)
+			(do_not_autoplace no)
+			(effects
+				(font
+					(size 1.27 1.27)
+				)
+				(justify left)
+			)
+		)
+		(property "Value" "FerriteBead"
+			(at 132.588 59.436 0)
+			(show_name no)
+			(do_not_autoplace no)
+			(effects
+				(font
+					(size 1.27 1.27)
+				)
+				(justify left)
+			)
+		)
+		(property "Footprint" ""
+			(at 144.272 58.42 90)
+			(hide yes)
+			(show_name no)
+			(do_not_autoplace no)
+			(effects
+				(font
+					(size 1.27 1.27)
+				)
+			)
+		)
+		(property "Datasheet" ""
+			(at 146.05 58.42 0)
+			(hide yes)
+			(show_name no)
+			(do_not_autoplace no)
+			(effects
+				(font
+					(size 1.27 1.27)
+				)
+			)
+		)
+		(property "Description" "Ferrite bead"
+			(at 146.05 58.42 0)
+			(hide yes)
+			(show_name no)
+			(do_not_autoplace no)
+			(effects
+				(font
+					(size 1.27 1.27)
+				)
+			)
+		)
+		(pin "1"
+		)
+		(pin "2"
+		)
+		(instances
+			(project "hs2-cdh-pcb"
+				(path "/e63e39d7-6ac0-4ffd-8aa3-1841a4541b55/4d115d59-e66a-4f9f-ab9e-2e7383353607"
+					(reference "FB3")
+					(unit 1)
+				)

Commit message: removing F from capacitors
Parts:
- C13, C14: value 0.1uF -> 0.1u
Changed lines of the file:
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@@
 			)
 		)
-		(property "Value" "0.1uF"
+		(property "Value" "0.1u"
 			(at 133.858 67.31 0)
 			(show_name no)
@@
 			)
 		)
-		(property "Value" "0.1uF"
+		(property "Value" "0.1u"
 			(at 161.29 67.3099 0)
 			(show_name no)

Commit message: Merge Payload and thermals
Parts:
- renumbered C14 to C58, C13 to C59, FB3 to FB4, U10 to U17
Changed lines of the file:
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@@
 		(dnp no)
 		(fields_autoplaced yes)
-		(property "Reference" "#PWR036"
+		(property "Reference" "#PWR0139"
 			(at 153.67 113.03 0)
 			(hide yes)
@@
 			(project "hs2-cdh-pcb"
 				(path "/e63e39d7-6ac0-4ffd-8aa3-1841a4541b55/4d115d59-e66a-4f9f-ab9e-2e7383353607"
-					(reference "#PWR036")
+					(reference "#PWR0139")
 					(unit 1)
 				)
@@
 		(in_pos_files yes)
 		(dnp no)
-		(property "Reference" "C14"
+		(property "Reference" "C58"
 			(at 133.858 64.77 0)
 			(show_name no)
@@
 			(project "hs2-cdh-pcb"
 				(path "/e63e39d7-6ac0-4ffd-8aa3-1841a4541b55/4d115d59-e66a-4f9f-ab9e-2e7383353607"
-					(reference "C14")
+					(reference "C58")
 					(unit 1)
 				)
@@
 		(dnp no)
 		(fields_autoplaced yes)
-		(property "Reference" "#PWR039"
+		(property "Reference" "#PWR0138"
 			(at 153.67 64.77 0)
 			(hide yes)
@@
 			(project "hs2-cdh-pcb"
 				(path "/e63e39d7-6ac0-4ffd-8aa3-1841a4541b55/4d115d59-e66a-4f9f-ab9e-2e7383353607"
-					(reference "#PWR039")
+					(reference "#PWR0138")
 					(unit 1)
 				)
@@
 		(dnp no)
 		(fields_autoplaced yes)
-		(property "Reference" "#PWR037"
+		(property "Reference" "#PWR0137"
 			(at 146.05 113.03 0)
 			(hide yes)
@@
 			(project "hs2-cdh-pcb"
 				(path "/e63e39d7-6ac0-4ffd-8aa3-1841a4541b55/4d115d59-e66a-4f9f-ab9e-2e7383353607"
-					(reference "#PWR037")
+					(reference "#PWR0137")
 					(unit 1)
 				)
@@
 		(dnp no)
 		(fields_autoplaced yes)
-		(property "Reference" "#PWR041"
+		(property "Reference" "#PWR0135"
 			(at 142.24 76.2 0)
 			(hide yes)
@@
 			(project "hs2-cdh-pcb"
 				(path "/e63e39d7-6ac0-4ffd-8aa3-1841a4541b55/4d115d59-e66a-4f9f-ab9e-2e7383353607"
-					(reference "#PWR041")
+					(reference "#PWR0135")
 					(unit 1)
 				)
@@
 		(dnp no)
 		(fields_autoplaced yes)
-		(property "Reference" "U10"
+		(property "Reference" "U17"
 			(at 155.8133 76.2 0)
 			(show_name no)
@@
 			(project "hs2-cdh-pcb"
 				(path "/e63e39d7-6ac0-4ffd-8aa3-1841a4541b55/4d115d59-e66a-4f9f-ab9e-2e7383353607"
-					(reference "U10")
+					(reference "U17")
 					(unit 1)
 				)
@@
 		(dnp no)
 		(fields_autoplaced yes)
-		(property "Reference" "#PWR038"
+		(property "Reference" "#PWR0140"
 			(at 157.48 76.2 0)
 			(hide yes)
@@
 			(project "hs2-cdh-pcb"
 				(path "/e63e39d7-6ac0-4ffd-8aa3-1841a4541b55/4d115d59-e66a-4f9f-ab9e-2e7383353607"
-					(reference "#PWR038")
+					(reference "#PWR0140")
 					(unit 1)
 				)
@@
 		(dnp no)
 		(fields_autoplaced yes)
-		(property "Reference" "#PWR040"
+		(property "Reference" "#PWR0136"
 			(at 146.05 58.42 0)
 			(hide yes)
@@
 			(project "hs2-cdh-pcb"
 				(path "/e63e39d7-6ac0-4ffd-8aa3-1841a4541b55/4d115d59-e66a-4f9f-ab9e-2e7383353607"
-					(reference "#PWR040")
+					(reference "#PWR0136")
 					(unit 1)
 				)
@@
 		(in_pos_files yes)
 		(dnp no)
-		(property "Reference" "FB3"
+		(property "Reference" "FB4"
 			(at 132.588 56.896 0)
 			(show_name no)
@@
 			(project "hs2-cdh-pcb"
 				(path "/e63e39d7-6ac0-4ffd-8aa3-1841a4541b55/4d115d59-e66a-4f9f-ab9e-2e7383353607"
-					(reference "FB3")
+					(reference "FB4")
 					(unit 1)
 				)
@@
 		(dnp no)
 		(fields_autoplaced yes)
-		(property "Reference" "C13"
+		(property "Reference" "C59"
 			(at 161.29 64.7699 0)
 			(show_name no)
@@
 			(project "hs2-cdh-pcb"
 				(path "/e63e39d7-6ac0-4ffd-8aa3-1841a4541b55/4d115d59-e66a-4f9f-ab9e-2e7383353607"
-					(reference "C13")
-					(unit 1)
-				)
+					(reference "C59")
+					(unit 1)
+				)
