File: sheets/storage.kicad_sch (KiCad schematic)
At the start: 15 parts, among them IC5 IS25LP01GJ-RMLE-TY, IC6 IS25LP01GJ-RMLE-TY, IC7 IS25LP01GJ-RMLE-TY, IC8 IS25LP01GJ-RMLE-TY, U11 ASFC64G31T5-51BIN

Commit message: removing F from capacitors
Parts:
- C10, C11, C12, C3, C4, C8, C9: value 0.1uF -> 0.1u
- C5, C7: value 4.7uF -> 4.7u
- C6: value 10uF -> 10u
Changed lines of the file:
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@@
 			)
 		)
-		(property "Value" "0.1uF"
+		(property "Value" "0.1u"
 			(at 20.32 71.1199 0)
 			(show_name no)
@@
 			)
 		)
-		(property "Value" "0.1uF"
+		(property "Value" "0.1u"
 			(at 177.8 41.9099 0)
 			(show_name no)
@@
 			)
 		)
-		(property "Value" "10uF"
+		(property "Value" "10u"
 			(at 171.45 27.9399 0)
 			(show_name no)
@@
 			)
 		)
-		(property "Value" "4.7uF"
+		(property "Value" "4.7u"
 			(at 165.1 41.9099 0)
 			(show_name no)
@@
 			)
 		)
-		(property "Value" "0.1uF"
+		(property "Value" "0.1u"
 			(at 20.32 36.8299 0)
 			(show_name no)
@@
 			)
 		)
-		(property "Value" "0.1uF"
+		(property "Value" "0.1u"
 			(at 20.32 106.6799 0)
 			(show_name no)
@@
 			)
 		)
-		(property "Value" "4.7uF"
+		(property "Value" "4.7u"
 			(at 184.15 27.9399 0)
 			(show_name no)
@@
 			)
 		)
-		(property "Value" "0.1uF"
+		(property "Value" "0.1u"
 			(at 20.32 140.9699 0)
 			(show_name no)
@@
 			)
 		)
-		(property "Value" "0.1uF"
+		(property "Value" "0.1u"
 			(at 196.85 27.9399 0)
 			(show_name no)
@@
 			)
 		)
-		(property "Value" "0.1uF"
+		(property "Value" "0.1u"
 			(at 127 71.1199 0)
 			(show_name no)

Commit message: Merge Payload and thermals
Parts:
- renumbered C9 to C1, C4 to C10, C10 to C2, C11 to C3, C12 to C4, C3 to C5, C7 to C6, C6 to C7, C5 to C9, IC5 to IC1, IC6 to IC2, IC7 to IC3, IC8 to IC4, U11 to U2
