File: hs2-cdh-pcb.kicad_sch (KiCad schematic)
At the start: 0 parts

Commit message: CDH Updated to have Payload USB interface and Trigger connectors
Other:
- added sheet Payload_USB (Payload_USB.kicad_sch)
Changed lines of the file:
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@@
+		)
+	)
+	(sheet
+		(at 16.002 115.062)
+		(size 54.102 39.878)
+		(exclude_from_sim no)
+		(in_bom yes)
+		(on_board yes)
+		(dnp no)
+		(fields_autoplaced yes)
+		(stroke
+			(width 0.1524)
+			(type solid)
+		)
+		(fill
+			(color 0 0 0 0)
+		)
+		(property "Sheetname" "Payload_USB"
+			(at 16.002 114.3504 0)
+			(show_name no)
+			(do_not_autoplace no)
+			(effects
+				(font
+					(size 1.27 1.27)
+				)
+				(justify left bottom)
+			)
+		)
+		(property "Sheetfile" "Payload_USB.kicad_sch"
+			(at 16.002 155.5246 0)
+			(show_name no)
+			(do_not_autoplace no)
+			(effects
+				(font
+					(size 1.27 1.27)
+				)
+				(justify left top)
+			)
+		)
+		(instances
+			(project "hs2-cdh-pcb"
+				(path "/e63e39d7-6ac0-4ffd-8aa3-1841a4541b55"
+					(page "7")
+				)
+			)
 		)
 	)

Commit message: Update
Other:
- added sheet Interfacing (Interfacing.kicad_sch)
Changed lines of the file:
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@@
+		)
+	)
+	(sheet
+		(at 78.994 115.57)
+		(size 49.53 39.624)
+		(exclude_from_sim no)
+		(in_bom yes)
+		(on_board yes)
+		(dnp no)
+		(fields_autoplaced yes)
+		(stroke
+			(width 0.1524)
+			(type solid)
+		)
+		(fill
+			(color 0 0 0 0)
+		)
+		(property "Sheetname" "Interfacing"
+			(at 78.994 114.8584 0)
+			(show_name no)
+			(do_not_autoplace no)
+			(effects
+				(font
+					(size 1.27 1.27)
+				)
+				(justify left bottom)
+			)
+		)
+		(property "Sheetfile" "Interfacing.kicad_sch"
+			(at 78.994 155.7786 0)
+			(hide yes)
+			(show_name no)
+			(do_not_autoplace no)
+			(effects
+				(font
+					(size 1.27 1.27)
+				)
+				(justify left top)
+			)
+		)
+		(instances
+			(project "hs2-cdh-pcb"
+				(path "/e63e39d7-6ac0-4ffd-8aa3-1841a4541b55"
+					(page "8")
+				)
+			)
 		)
 	)
