File: hs2-cdh-pcb.kicad_sch (KiCad schematic)
At the start: 0 parts

Commit message: pushing storage
Other:
- sheet nor_flash.kicad_sch renamed storage
- added sheet ADCS sun ADC (sheets/adcs_sun_adc.kicad_sch)
- sheet storage: file sheets/nor_flash.kicad_sch -> sheets/storage.kicad_sch
Changed lines of the file:
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@@
+	)
+	(sheet
+		(at 15.24 115.57)
+		(size 49.53 33.02)
+		(exclude_from_sim no)
+		(in_bom yes)
+		(on_board yes)
+		(dnp no)
+		(fields_autoplaced yes)
+		(stroke
+			(width 0.1524)
+			(type solid)
+		)
+		(fill
+			(color 0 0 0 0)
+		)
+		(property "Sheetname" "ADCS sun ADC"
+			(at 15.24 114.8584 0)
+			(show_name no)
+			(do_not_autoplace no)
+			(effects
+				(font
+					(size 1.27 1.27)
+				)
+				(justify left bottom)
+			)
+		)
+		(property "Sheetfile" "sheets/adcs_sun_adc.kicad_sch"
+			(at 15.24 149.1746 0)
+			(show_name no)
+			(do_not_autoplace no)
+			(effects
+				(font
+					(size 1.27 1.27)
+				)
+				(justify left top)
+			)
+		)
+		(instances
+			(project "hs2-cdh-pcb"
+				(path "/e63e39d7-6ac0-4ffd-8aa3-1841a4541b55"
+					(page "8")
+				)
+			)
+		)
 	)
 	(sheet
@@
 	)
 	(sheet
-		(at 175.26 22.86)
-		(size 80.01 139.7)
+		(at 121.92 17.78)
+		(size 54.61 46.99)
 		(exclude_from_sim no)
 		(in_bom yes)
@@
 			(color 0 0 0 0)
 		)
-		(property "Sheetname" "nor_flash.kicad_sch"
-			(at 175.26 22.1484 0)
+		(property "Sheetname" "storage"
+			(at 121.92 17.0684 0)
 			(show_name no)
 			(do_not_autoplace no)
@@
 			)
 		)
-		(property "Sheetfile" "sheets/nor_flash.kicad_sch"
-			(at 175.26 163.1446 0)
+		(property "Sheetfile" "sheets/storage.kicad_sch"
+			(at 121.92 65.3546 0)
 			(show_name no)
 			(do_not_autoplace no)

Commit message: adding pc104 from EPS
Other:
- sheet ADCS sun ADC renamed ACDS sun ADC
Changed lines of the file:
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@@
 			(color 0 0 0 0)
 		)
-		(property "Sheetname" "ADCS sun ADC"
+		(property "Sheetname" "ACDS sun ADC"
 			(at 15.24 114.8584 0)
 			(show_name no)

Commit message: Merge Payload and thermals
Other:
- added sheet Interfacing (sheets\Interfacing.kicad_sch)
- added sheet Payload (sheets\Payload_USB.kicad_sch)
Changed lines of the file:
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@@
+	)
+	(sheet
+		(at 76.708 117.856)
+		(size 48.26 26.162)
+		(exclude_from_sim no)
+		(in_bom yes)
+		(on_board yes)
+		(dnp no)
+		(fields_autoplaced yes)
+		(stroke
+			(width 0.1524)
+			(type solid)
+		)
+		(fill
+			(color 0 0 0 0)
+		)
+		(property "Sheetname" "Payload"
+			(at 76.708 117.1444 0)
+			(show_name no)
+			(do_not_autoplace no)
+			(effects
+				(font
+					(size 1.27 1.27)
+				)
+				(justify left bottom)
+			)
+		)
+		(property "Sheetfile" "sheets\\Payload_USB.kicad_sch"
+			(at 76.708 144.6026 0)
+			(show_name no)
+			(do_not_autoplace no)
+			(effects
+				(font
+					(size 1.27 1.27)
+				)
+				(justify left top)
+			)
+		)
+		(instances
+			(project "hs2-cdh-pcb"
+				(path "/e63e39d7-6ac0-4ffd-8aa3-1841a4541b55"
+					(page "7")
+				)
+			)
+		)
 	)
 	(sheet
@@
 				)
 			)
+		)
+	)
+	(sheet
+		(at 15.748 159.258)
+		(size 50.546 32.258)
+		(exclude_from_sim no)
+		(in_bom yes)
+		(on_board yes)
+		(dnp no)
+		(fields_autoplaced yes)
+		(stroke
+			(width 0.1524)
+			(type solid)
+		)
+		(fill
+			(color 0 0 0 0)
+		)
+		(property "Sheetname" "Interfacing"
+			(at 15.748 158.5464 0)
+			(show_name no)
+			(do_not_autoplace no)
+			(effects
+				(font
+					(size 1.27 1.27)
+				)
+				(justify left bottom)
+			)
+		)
+		(property "Sheetfile" "sheets\\Interfacing.kicad_sch"
+			(at 15.748 192.1006 0)
+			(show_name no)
+			(do_not_autoplace no)
+			(effects
+				(font
+					(size 1.27 1.27)
+				)
+				(justify left top)
+			)
+		)
+		(instances
+			(project "hs2-cdh-pcb"
+				(path "/e63e39d7-6ac0-4ffd-8aa3-1841a4541b55"
+					(page "9")
+				)
+			)
